File: schematic/dj-console/mixer.kicad_sch (KiCad schematic)
At the start: 0 parts

Commit message: Created first version of mixer circuit and added tempo sliders on decks
Parts:
- added C39, C41, C42, C43, C44, C73: C, symbol Device:C
- added C40, C45, C46, C47, C48, C49, C50, C75, C76: 10uF, symbol Device:C_Polarized
- added C51, C52: 1uF, symbol Device:C_Polarized
- added C71: 1nF, symbol Device:C
- added D53: D, symbol Device:D
- added D55: LED, symbol Device:LED
- added DECK_FADER1, EQ_FX1_1, EQ_FX2_1, EQ_HIGH1, EQ_LOW1, EQ_MID1: 100kOhm, symbol Device:R_Potentiometer
- added HEADPHOONES_SW1: SW_Push, symbol Switch:SW_Push
- added Q27: BC547, Package_TO_SOT_THT:TO-92_Inline, symbol Transistor_BJT:BC547
- added R105, R106, R107, R108, R109, R110, R111, R112, R113, R114, R133, R138: R, symbol Device:R
- added R129: 43kOhm, symbol Device:R
- added R130: 100kOhm, symbol Device:R
- added R134: 12kOhm, symbol Device:R
- added R137: 510Ohm, symbol Device:R
- added U17, U18, U19, U20, U21, U35: LM741, symbol Amplifier_Operational:LM741
- added U22, U23: MCP3204, symbol Analog_ADC:MCP3204
- added U33: (no value), symbol D-flipflop:CD4013B
Connections:
- new net: EQ_FX1_1.2, R108.1
- new net: C43.2, R108.2, R113.1, U20.2 (-)
- new net: D55.1 (K), Q27.1 (C)
- new net: Q27.2 (B), R129.2
- new net: C73.2, R133.2, R138.1, U35.2 (-)
- new net: DECK_FADER1.2, R133.1
- new net: C39.2, R105.2, R110.1, U17.2 (-)
- new net: D55.2 (A), R137.2
- new net: C41.2, R106.2, R111.1, U18.2 (-)
- new net: C42.2, R107.2, R112.1, U19.2 (-)
- new net: EQ_LOW1.2, R107.1
- new net: D53.2 (A), HEADPHOONES_SW1.1, R130.1, R134.1
- new net: C44.2, R109.2, R114.1, U21.2 (-)
- new net: EQ_MID1.2, R106.1
- new net: EQ_HIGH1.2, R105.1
- new net: EQ_FX2_1.2, R109.1
- new net +12V: C40.1, C45.1, C46.1, C47.1, C48.1, C75.1, R137.1, U17.7 (V+), U18.7 (V+), U19.7 (V+), U20.7 (V+), U21.7 (V+), U35.7 (V+)
- new net +5V: C49.1, C50.1, C51.1, C52.1, C76.1, DECK_FADER1.1, EQ_FX1_1.1, EQ_FX2_1.1, EQ_HIGH1.1, EQ_LOW1.1, EQ_MID1.1, HEADPHOONES_SW1.2, U22.13 (Vref), U22.14 (Vdd), U23.13 (Vref), U23.14 (Vdd), U33.14 (VDD)
- new net DECK_FADER_filtered: C73.1, R138.2, U23.2 (CH1), U35.6
- new net EQ_FX1_filtered: C43.1, R113.2, U20.6, U22.4 (CH3)
- new net EQ_FX2_filtered: C44.1, R114.2, U21.6, U23.1 (CH0)
- new net EQ_HIGH_filtered: C39.1, R110.2, U17.6, U22.1 (CH0)
- new net EQ_LOW_filtered: C42.1, R112.2, U19.6, U22.3 (CH2)
- new net EQ_MID_filtered: C41.1, R111.2, U18.6, U22.2 (CH1)
- new net GND: C40.2, C45.2, C46.2, C47.2, C48.2, C49.2, C50.2, C51.2, C52.2, C71.2, C75.2, C76.2, DECK_FADER1.3, EQ_FX1_1.3, EQ_FX2_1.3, EQ_HIGH1.3, EQ_LOW1.3, EQ_MID1.3, Q27.3 (E), R130.2, U17.3 (+), U17.4 (V-), U18.3 (+), U18.4 (V-), U19.3 (+), U19.4 (V-), U20.3 (+), U20.4 (V-), U21.3 (+), U21.4 (V-), U22.12 (AGND), U22.7 (DGND), U23.12 (AGND), U23.7 (DGND), U33.7 (VSS), U35.3 (+), U35.4 (V-)
- new net HEADPHONES_STAT: R129.1, U33.1 (Q1)
- new net HEADPHONES_SW: C71.1, D53.1 (K), R134.2, U33.3 (CLK1)
- new net TEMPO_SLIDER_filtered: U23.3 (CH2)
- new net ~{HEADPHONES_LED}: U33.2 (~{Q1}), U33.5 (D1)
- no-connect marks 0 -> 18

Commit message: Added MASTER and HEADPHONES gain together with crossfader slider
Connections:
- no-connect marks 18 -> 17
Changed lines of the file:
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@@
+	)
+	(junction
+		(at 552.45 96.52)
+		(diameter 0)
+		(color 0 0 0 0)
 	)
 	(junction
@@
 		(color 0 0 0 0)
 	)
+	(junction
+		(at 543.56 96.52)
+		(diameter 0)
+		(color 0 0 0 0)
+	)
 	(no_connect
 		(at 72.39 382.27)
@@
 	)
 	(no_connect
-		(at 525.78 167.64)
-	)
-	(no_connect
 		(at 72.39 133.35)
 	)
@@
 	(wire
 		(pts
+			(xy 552.45 96.52) (xy 556.26 96.52)
+		)
+		(stroke
+			(width 0)
+			(type default)
+		)
+	)
+	(wire
+		(pts
 			(xy 556.26 241.3) (xy 556.26 261.62)
 		)
@@
 	(wire
 		(pts
+			(xy 552.45 133.35) (xy 552.45 96.52)
+		)
+		(stroke
+			(width 0)
+			(type default)
+		)
+	)
+	(wire
+		(pts
 			(xy 58.42 292.1) (xy 58.42 309.88)
 		)
@@
 	(wire
 		(pts
-			(xy 543.56 96.52) (xy 561.34 96.52)
+			(xy 533.4 96.52) (xy 543.56 96.52)
 		)
 		(stroke
@@
 	(wire
 		(pts
+			(xy 502.92 133.35) (xy 552.45 133.35)
+		)
+		(stroke
+			(width 0)
+			(type default)
+		)
+	)
+	(wire
+		(pts
 			(xy 68.58 226.06) (xy 68.58 231.14)
 		)
@@
 	(wire
 		(pts
-			(xy 494.03 177.8) (xy 511.81 177.8)
+			(xy 502.92 177.8) (xy 511.81 177.8)
 		)
 		(stroke
@@
 	(wire
 		(pts
+			(xy 543.56 96.52) (xy 552.45 96.52)
+		)
+		(stroke
+			(width 0)
+			(type default)
+		)
+	)
+	(wire
+		(pts
 			(xy 74.93 146.05) (xy 74.93 151.13)
 		)
@@
 	(wire
 		(pts
-			(xy 158.75 132.08) (xy 142.24 132.08)
+			(xy 158.75 132.08) (xy 138.43 132.08)
 		)
 		(stroke
@@
 		(pts
 			(xy 69.85 354.33) (xy 69.85 367.03)
+		)
+		(stroke
+			(width 0)
+			(type default)
+		)
+	)
+	(wire
+		(pts
+			(xy 502.92 177.8) (xy 502.92 133.35)
 		)
 		(stroke
@@
 		)
 	)
-	(label "HEADPHONES_LED"
-		(at 494.03 177.8 0)
+	(label "EQ_FX2_filtered"
+		(at 138.43 132.08 0)
 		(effects
 			(font
@@
 			)
 			(justify left bottom)
-		)
-	)
-	(label "EQ_FX2_filtered"
-		(at 142.24 132.08 0)
-		(effects
-			(font
-				(size 1.27 1.27)
-			)
-			(justify left bottom)
-		)
-	)
-	(label "HEADPHONES_LED"
-		(at 561.34 96.52 180)
-		(effects
-			(font
-				(size 1.27 1.27)
-			)
-			(justify right bottom)
 		)
 	)
@@
 	(hierarchical_label "HEADPHONES_STAT"
 		(shape output)
-		(at 561.34 96.52 0)
+		(at 556.26 96.52 0)
 		(effects
 			(font

Commit message: Changed filtering circuit for knobs
Parts:
- removed C40, C75: 10uF, symbol Device:C_Polarized
- removed C73: C, symbol Device:C
- removed R106, R108, R111, R112, R114, R133, R138: R, symbol Device:R
- removed U35: LM741, symbol Amplifier_Operational:LM741
- added C40, C55: 4.7nF, symbol Device:C
- added C49, C50, C87: 0.1uF, symbol Device:C_Polarized
- added DECK_GAIN1: 10kOhm, symbol Device:R_Potentiometer
- added R115, R83: 8.2kOhm, symbol Device:R
- added U22, U41: LM741, symbol Amplifier_Operational:LM741
- C39, C41, C42, C43, C44: value C -> 4.7nF
- C45, C46, C47, C48: value 10uF -> 0.1uF
- C88: renamed from C76; value 10uF -> 0.1uF
- DECK_FADER1, EQ_FX1_1, EQ_FX2_1, EQ_HIGH1, EQ_LOW1, EQ_MID1: value 100kOhm -> 10kOhm
- R105, R107, R109, R110, R113: value R -> 8.2kOhm
- renumbered C49 to C51, C50 to C52, C51 to C53, C52 to C54, C71 to C56, R129 to R116, R130 to R117, R134 to R118, R137 to R123, U22 to U23, U23 to U24, U33 to U25
Connections:
- net +12V: now also C49.1, C50.1, C87.1, U22.7 (V+), U41.7 (V+)
- net +5V: now also DECK_GAIN1.1
- net DECK_FADER_filtered: now also U41.2 (-), U41.6
- net EQ_FX1_filtered: now also U20.2 (-); no longer C43.1, R113.2
- net EQ_FX2_filtered: now also U21.2 (-); no longer C44.1
- net EQ_HIGH_filtered: no longer C39.1, R110.2, U17.6
- net EQ_LOW_filtered: now also U19.2 (-); no longer C42.1
- net EQ_MID_filtered: now also U17.2 (-), U17.6, U18.2 (-); no longer C41.1
- net GND: now also C39.2, C41.2, C42.2, C43.2, C44.2, C40.2, C49.2, C50.2, C55.2, C87.2, DECK_GAIN1.3, U22.4 (V-), U41.4 (V-); no longer U17.3 (+), U18.3 (+), U19.3 (+), U20.3 (+), U21.3 (+)
- net TEMPO_SLIDER_filtered: now also U24.4 (CH3); no longer U24.3 (CH2)
- net at EQ_FX1_1.2: now also R109.1
- net at DECK_FADER1.2: now also R115.1
- net at EQ_MID1.2: now also R105.1
- net at EQ_HIGH1.2: now also R83.1; no longer R105.1
- net at EQ_FX2_1.2: now also R110.1; no longer R109.1
- new net: C41.1, R107.2, U19.3 (+)
- new net: C42.1, R109.2, U20.3 (+)
- new net: C55.1, R115.2, U41.3 (+)
- new net: C39.1, R83.2, U17.3 (+)
- new net: C40.1, R105.2, U18.3 (+)
- new net: C44.1, R113.2, U22.3 (+)
- new net: C43.1, R110.2, U21.3 (+)
- new net: DECK_GAIN1.2, R113.1
- new net DECK_GAIN_filtered: U22.2 (-), U22.6, U24.3 (CH2)
- no-connect marks 17 -> 18

Commit message: Added I2C and SPI busses
Parts:
- added C87: 1nF, symbol Device:C
- added D55: D, symbol Device:D
- added R118: 100kOhm, symbol Device:R
- added R132: 12kOhm, symbol Device:R
- added TRACK_LOAD_SW1: SW_Push, symbol Switch:SW_Push
- renumbered C87 to C88, C88 to C91, D55 to D57, HEADPHOONES_SW1 to HEADPHONES_SW1, R118 to R123, R123 to R133
Connections:
- net +5V: now also TRACK_LOAD_SW1.2
- net GND: now also C87.2, R118.2
- net ADC_SPI.MISO: now reaches U23.10 (Dout)
- net ADC_SPI.MISO: now also U24.10 (Dout)
- net ADC_SPI.CLK: now reaches U23.11 (CLK)
- net ADC_SPI.CLK: now also U24.11 (CLK)
- net ADC_SPI.MOSI: now reaches U23.9 (Din)
- net ADC_SPI.MOSI: now also U24.9 (Din)
- new net: D55.2 (A), R118.1, R132.1, TRACK_LOAD_SW1.1
- new net TRACK_LOAD_SW: C87.1, D55.1 (K), R132.2
Other:
- moved on the sheet: C55, C88, C91, D57, DECK_FADER1, Q27, R115, R116, R133, U25
